File: amp_schematic.brd (EAGLE design)
At the start: 60 x 60 mm, 22 parts, among them J1 DCJ0202, U1 OPA2132PA

Commit message: made some changes
yo diggity
Parts:
- renumbered U$1 to VOL, U$2 to OUTPUT, U1 to OPAMP
Routing:
- net N$13: track 32.7 -> 37.6 mm
- net N$15: track 37.2 -> 38.6 mm, vias 0 -> 1
- net N$12: track 48.1 -> 48.7 mm, vias 2 -> 1
- added copper zone on layer 16, net GND
