File: amp_schematic.sch (EAGLE design)
At the start: 22 parts, among them J1 DCJ0202, U1 OPA2132PA

Commit message: made some changes
yo diggity
Parts:
- renumbered U$1 to VOL, U$2 to OUTPUT, U1 to OPAMP
